File: kicad/benboard.kicad_sch (KiCad schematic)
At the start: 60 parts, among them J1 USB_C_Receptacle_USB2.0, J3 Conn_ARM_SWD_TagConnect_TC203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, SW1 SW_Push, U1 nRF52840, U2 BQ24075RGT, Y1 32MHz, Y2 32.768kHz

Commit message: routes for some stuff
Parts:
- added J4: Conn_01x02_Pin, Connector_JST:JST_EH_B2B-EH-A_1x02_P2.50mm_Vertical, symbol Connector:Conn_01x02_Pin
- added J5: Conn_Coaxial, Connector_Coaxial:SMA_Amphenol_132134-10_Vertical, symbol Connector:Conn_Coaxial
- added SW22: SW_Push, Button_Switch_SMD:SW_SPST_CK_KXT3, symbol Switch:SW_Push
Connections:
- net ANTENNA: now also J5.1 (In); no longer C14.1, L4.1
- net GND: now also J4.2 (Pin_2), SW22.1
- net RST: now also SW22.2
- net VBAT: now also J4.1 (Pin_1)
- new net: C14.1, J5.2 (Ext), L4.1
Changed lines of the file:
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@@
     (stroke (width 0) (type default))
   )
+  (wire (pts (xy 27.94 185.42) (xy 27.94 186.69))
+    (stroke (width 0) (type default))
+  )
   (wire (pts (xy 116.84 179.07) (xy 115.57 179.07))
     (stroke (width 0) (type default))
@@
     (stroke (width 0) (type default))
   )
-  (wire (pts (xy 33.02 102.87) (xy 34.29 102.87))
-    (stroke (width 0) (type default))
-  )
   (wire (pts (xy 48.26 194.31) (xy 49.53 194.31))
     (stroke (width 0) (type default))
@@
     (stroke (width 0) (type default))
   )
+  (wire (pts (xy 218.44 31.75) (xy 218.44 30.48))
+    (stroke (width 0) (type default))
+  )
   (wire (pts (xy 115.57 201.93) (xy 116.84 201.93))
     (stroke (width 0) (type default))
@@
     (stroke (width 0) (type default))
   )
+  (wire (pts (xy 33.02 102.87) (xy 34.29 102.87))
+    (stroke (width 0) (type default))
+  )
   (wire (pts (xy 62.23 77.47) (xy 62.23 73.66))
     (stroke (width 0) (type default))
@@
     (stroke (width 0) (type default))
   )
+  (wire (pts (xy 39.37 185.42) (xy 40.64 185.42))
+    (stroke (width 0) (type default))
+  )
+  (wire (pts (xy 217.17 27.94) (xy 218.44 27.94))
+    (stroke (width 0) (type default))
+  )
   (wire (pts (xy 271.78 63.5) (xy 270.51 63.5))
     (stroke (width 0) (type default))
@@
     (stroke (width 0) (type default))
   )
+  (wire (pts (xy 27.94 109.22) (xy 27.94 107.95))
+    (stroke (width 0) (type default))
+  )
   (wire (pts (xy 115.57 191.77) (xy 116.84 191.77))
     (stroke (width 0) (type default))
@@
     (stroke (width 0) (type default))
   )
+  (wire (pts (xy 27.94 185.42) (xy 29.21 185.42))
+    (stroke (width 0) (type default))
+  )
   (wire (pts (xy 85.09 41.91) (xy 85.09 46.99))
     (stroke (width 0) (type default))
@@
     (stroke (width 0) (type default))
   )
+  (wire (pts (xy 217.17 30.48) (xy 218.44 30.48))
+    (stroke (width 0) (type default))
+  )
   (wire (pts (xy 35.56 143.51) (xy 43.18 143.51))
     (stroke (width 0) (type default))
@@
     )
   )
-  (global_label "ANTENNA" (shape input) (at 33.02 102.87 90) (fields_autoplaced)
-    (effects (font (size 1.27 1.27)) (justify left))
-    (property "Intersheetrefs" "${INTERSHEET_REFS}" (at 33.02 91.5995 90)
-      (effects (font (size 1.27 1.27)) (justify left) hide)
+  (global_label "ANTENNA" (shape input) (at 27.94 109.22 270) (fields_autoplaced)
+    (effects (font (size 1.27 1.27)) (justify right))
+    (property "Intersheetrefs" "${INTERSHEET_REFS}" (at 27.94 120.4905 90)
+      (effects (font (size 1.27 1.27)) (justify right) hide)
     )
   )
@@
     )
   )
+  (global_label "VBAT" (shape input) (at 218.44 27.94 0) (fields_autoplaced)
+    (effects (font (size 1.27 1.27)) (justify left))
+    (property "Intersheetrefs" "${INTERSHEET_REFS}" (at 225.84 27.94 0)
+      (effects (font (size 1.27 1.27)) (justify left) hide)
+    )
+  )
   (global_label "SDA" (shape input) (at 176.53 185.42 180) (fields_autoplaced)
     (effects (font (size 1.27 1.27)) (justify right))
@@
     )
   )
+  (global_label "RST" (shape input) (at 40.64 185.42 0) (fields_autoplaced)
+    (effects (font (size 1.27 1.27)) (justify left))
+    (property "Intersheetrefs" "${INTERSHEET_REFS}" (at 47.0723 185.42 0)
+      (effects (font (size 1.27 1.27)) (justify left) hide)
+    )
+  )
   (global_label "VDDH" (shape input) (at 176.53 180.34 180) (fields_autoplaced)
     (effects (font (size 1.27 1.27)) (justify right))
@@
     )
   )
+  (symbol (lib_id "Switch:SW_Push") (at 34.29 185.42 0) (unit 1)
+    (in_bom yes) (on_board yes) (dnp no) (fields_autoplaced)
+    (property "Reference" "SW22" (at 34.29 177.8 0)
+      (effects (font (size 1.27 1.27)))
+    )
+    (property "Value" "SW_Push" (at 34.29 180.34 0)
+      (effects (font (size 1.27 1.27)))
+    )
+    (property "Footprint" "Button_Switch_SMD:SW_SPST_CK_KXT3" (at 34.29 180.34 0)
+      (effects (font (size 1.27 1.27)) hide)
+    )
+    (property "Datasheet" "~" (at 34.29 180.34 0)
+      (effects (font (size 1.27 1.27)) hide)
+    )
+    (pin "1")
+    (pin "2")
+    (instances
+      (project "benboard"
+        (path "/b2065370-6f3a-4205-b26a-a9c2368077cd"
+          (reference "SW22") (unit 1)
+        )
+      )
+    )
+  )
   (symbol (lib_id "power:GND") (at 200.66 127 0) (unit 1)
     (in_bom yes) (on_board yes) (dnp no)
@@
     )
   )
+  (symbol (lib_id "power:GND") (at 27.94 186.69 0) (unit 1)
+    (in_bom yes) (on_board yes) (dnp no)
+    (property "Reference" "#PWR048" (at 27.94 193.04 0)
+      (effects (font (size 1.27 1.27)) hide)
+    )
+    (property "Value" "GND" (at 27.94 190.5 0)
+      (effects (font (size 1.27 1.27)))
+    )
+    (property "Footprint" "" (at 27.94 186.69 0)
+      (effects (font (size 1.27 1.27)) hide)
+    )
+    (property "Datasheet" "" (at 27.94 186.69 0)
+      (effects (font (size 1.27 1.27)) hide)
+    )
+    (pin "1")
+    (instances
+      (project "benboard"
+        (path "/b2065370-6f3a-4205-b26a-a9c2368077cd"
+          (reference "#PWR048") (unit 1)
+        )
+      )
+    )
+  )
   (symbol (lib_id "Switch:SW_Push") (at 229.87 115.57 0) (unit 1)
     (in_bom yes) (on_board yes) (dnp no)
@@
     )
   )
+  (symbol (lib_id "Connector:Conn_01x02_Pin") (at 212.09 27.94 0) (unit 1)
+    (in_bom yes) (on_board yes) (dnp no) (fields_autoplaced)
+    (property "Reference" "J4" (at 212.725 22.86 0)
+      (effects (font (size 1.27 1.27)))
+    )
+    (property "Value" "Conn_01x02_Pin" (at 212.725 25.4 0)
+      (effects (font (size 1.27 1.27)))
+    )
+    (property "Footprint" "Connector_JST:JST_EH_B2B-EH-A_1x02_P2.50mm_Vertical" (at 212.09 27.94 0)
+      (effects (font (size 1.27 1.27)) hide)
+    )
+    (property "Datasheet" "~" (at 212.09 27.94 0)
+      (effects (font (size 1.27 1.27)) hide)
+    )
+    (pin "1")
+    (pin "2")
+    (instances
+      (project "benboard"
+        (path "/b2065370-6f3a-4205-b26a-a9c2368077cd"
+          (reference "J4") (unit 1)
+        )
+      )
+    )
+  )
   (symbol (lib_id "Device:C") (at 208.28 58.42 0) (unit 1)
     (in_bom yes) (on_board yes) (dnp no)
@@
     )
   )
+  (symbol (lib_id "power:GND") (at 218.44 31.75 0) (unit 1)
+    (in_bom yes) (on_board yes) (dnp no)
+    (property "Reference" "#PWR047" (at 218.44 38.1 0)
+      (effects (font (size 1.27 1.27)) hide)
+    )
+    (property "Value" "GND" (at 218.44 35.56 0)
+      (effects (font (size 1.27 1.27)))
+    )
+    (property "Footprint" "" (at 218.44 31.75 0)
+      (effects (font (size 1.27 1.27)) hide)
+    )
+    (property "Datasheet" "" (at 218.44 31.75 0)
+      (effects (font (size 1.27 1.27)) hide)
+    )
+    (pin "1")
+    (instances
+      (project "benboard"
+        (path "/b2065370-6f3a-4205-b26a-a9c2368077cd"
+          (reference "#PWR047") (unit 1)
+        )
+      )
+    )
+  )
   (symbol (lib_id "Switch:SW_Push") (at 207.01 125.73 0) (unit 1)
     (in_bom yes) (on_board yes) (dnp no)
@@
         )
       )
+    )
+  )
+  (symbol (lib_id "Connector:Conn_Coaxial") (at 27.94 102.87 90) (unit 1)
+    (in_bom yes) (on_board yes) (dnp no) (fields_autoplaced)
+    (property "Reference" "J5" (at 28.2332 96.52 90)
+      (effects (font (size 1.27 1.27)))
+    )
+    (property "Value" "Conn_Coaxial" (at 28.2332 99.06 90)
+      (effects (font (size 1.27 1.27)))
+    )
+    (property "Footprint" "Connector_Coaxial:SMA_Amphenol_132134-10_Vertical" (at 27.94 102.87 0)
+      (effects (font (size 1.27 1.27)) hide)
+    )
+    (property "Datasheet" " ~" (at 27.94 102.87 0)
+      (effects (font (size 1.27 1.27)) hide)
+    )
+    (pin "1")
+    (pin "2")
+    (instances
+      (project "benboard"
+        (path "/b2065370-6f3a-4205-b26a-a9c2368077cd"
+          (reference "J5") (unit 1)
+        )
+      )

Commit message: VIK Compatible
Connections:
- net MISO: now also U1.A14 (P1.15); no longer U1.B15 (P1.14)
- net MOSI: now also U1.A20 (P1.10); no longer U1.B17 (P1.12)
- net SCL: now also U1.B17 (P1.12); no longer U1.B19 (P1.11)
- net SCLK: now also U1.A10 (AIN5/P0.29); no longer U1.A14 (P1.15)
- net SDA: now also U1.B19 (P1.11); no longer U1.A20 (P1.10)
- net VIK_RGB: now also U1.B15 (P1.14); no longer U1.G1 (P0.26)

Commit message: proper footprint
Parts:
- J5: footprint Connector_Coaxial:SMA_Amphenol_132134-10_Vertical -> Connector_Coaxial:U.FL_Hirose_U.FL-R-SMT-1_Vertical
Changed lines of the file:
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@@
       (effects (font (size 1.27 1.27)))
     )
-    (property "Footprint" "Connector_Coaxial:SMA_Amphenol_132134-10_Vertical" (at 27.94 102.87 0)
+    (property "Footprint" "Connector_Coaxial:U.FL_Hirose_U.FL-R-SMT-1_Vertical" (at 27.94 102.87 0)
       (effects (font (size 1.27 1.27)) hide)
     )
