File: kicad/benboard.kicad_sch (KiCad schematic)
At the start: 63 parts, among them J1 USB_C_Receptacle_USB2.0, J3 Conn_ARM_SWD_TagConnect_TC203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, J4 Conn_01x02_Pin, J5 Conn_Coaxial, SW1 SW_Push, SW22 SW_Push, U1 nRF52840, U2 BQ24075RGT, Y1 32MHz, Y2 32.768kHz

Commit message: this is so epic
Parts:
- removed R1, R2: 5.1k, Resistor_SMD:R_0603_1608Metric, symbol Device:R
- added U3: nPM1300-QEXX, Package_DFN_QFN:QFN-32-1EP_5x5mm_P0.5mm_EP3.6x3.6mm_ThermalVias, symbol nrf-npm:nPM1300-QEXX
Connections:
- net RST: now also U3.7 (GPIO0)
- net SDA: now also U1.J1 (AIN2/P0.04), U3.13 (SDA); no longer J2.3 (SDA), U1.B19 (P1.11)
- net VBAT: now also U3.19 (VBAT)
- net VBUS: now also U3.21 (VBUS)
- net CC1: now reaches J1.A5 (CC1)
- net CC1: now also U3.23 (CC1)
- net CC2: now reaches J1.B5 (CC2)
- net CC2: now also U3.24 (CC2)
- net SCK: now reaches U1.K2 (AIN3/P0.05)
- net SCK: now also U3.14 (SCL)
- net SCL renamed VIK_SCL
- new net: U3.2 (PVSS1), U3.33 (AVSS), U3.6 (PVSS2)
- new net VIK_SDA: J2.3 (SDA), U1.B19 (P1.11)
Other:
- note added: "(global_label "VCC1" (shape input) (at 269.24 237.49 0) (fields_autoplaced) (effects (font (size 1.27 1.27)) (justify left)) (uuid 764a8019-8547-4c42-bd1d-b73854bda07f) (property "Intersheetrefs" "${INTERSHEET_REFS}" (at 277.0633 237.49 0) (effects (font (size 1.27 1.27)) (justify left) hide) ) ) (global_label "VCC1" (shape input) (at 269.24 237.49 0) (fields_autoplaced) (effects (font (size 1.27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"
- note added: "Power Management"
- note added: "[x] Optional 32kHz on X1/2 [x] Figure out VDD [-] IC for power management [ ] i2c pullups [x] SWD [x] VIK [-] RESET / POWER BUTTON [ ] ESD PROTECTION [ ] BETTER POWER CIRCUITRY (In1.Cu = 3v3 ?) [x] BATTERY PADS [x] PROBE POINTS [-] ANT JUMPERS"
- note removed: "Battery Charging"
- note removed: "[x] Optional 32kHz on X1/2 [ ] Figure out VDD"
- moved on the sheet: C1, C10, C11, C12, C13, C14, C16, C17, C18, C19, C2, C20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

Commit message: schematic basically done
Parts:
- removed R3, R4, R5: 10k, Resistor_SMD:R_0603_1608Metric, symbol Device:R
- removed RED1: LED, LED_SMD:LED_0805_2012Metric, symbol Device:LED
- removed U2: BQ24075RGT, Package_DFN_QFN:VQFN-16-1EP_3x3mm_P0.5mm_EP1.6x1.6mm, symbol Battery_Management:BQ24075RGT
- added C15: 1uF, Capacitor_SMD:C_0603_1608Metric, symbol Device:C
- added C24, C26: 100nF, Capacitor_SMD:C_0603_1608Metric, symbol Device:C
- added C25: 10uF, Capacitor_SMD:C_0603_1608Metric, symbol Device:C
- added C27: 2.2uF, Capacitor_SMD:C_0603_1608Metric, symbol Device:C
- added D1, D2, D3: LED, symbol Device:LED
- added D4: PRTR5V0U2X, Package_TO_SOT_SMD:SOT-143, symbol Power_Protection:PRTR5V0U2X
- added L5: 4.7uH, symbol Device:L
- added L6, L7: 2.2uH, symbol Device:L
- added R1: 47k, symbol Device:R
- added R2: 250k, symbol Device:R
- added TH1: Thermistor, symbol Device:Thermistor
- added U2: TPS61222DCK, Package_TO_SOT_SMD:Texas_R-PDSO-G6, symbol Regulator_Switching:TPS61222DCK
- C1: value 4.7uF -> 1uF
- C18: value 1uF -> 10uF
- C19, C20: value 4.7uF -> 10uF
Connections:
- net VDD_NRF is gone; now on net +1V8: C10.1, C11.1, C12.1, C13.1, C9.1, L3.2, U1.A22 (VDD), U1.AD14 (VDD), U1.AD23 (VDD), U1.B1 (VDD), U1.W1 (VDD)
- net D+: now also D4.2 (I/O1)
- net D-: now also D4.3 (I/O2)
- net GND: now also U3.15 (SHPHLD), U3.2 (PVSS1), U3.33 (AVSS), U3.6 (PVSS2), C15.2, C24.2, C25.2, C26.2, C27.2, D4.1 (GND), R1.2, R2.1, TH1.1, U2.3 (GND)
- net VBAT: now also C27.1; no longer C20.1
- net +1V8: now reaches U3.1 (VOUT1)
- net +1V8: now also C2.1, C20.1, U1.Y2 (VDDH), U3.12 (VDDIO), C26.1, L6.1
- net at U3.16 (VSET2): now also R2.2
- net at U3.17 (VSET1): now also R1.1
- net at U3.18 (NTC): now also TH1.2
- net VSYS: now reaches U3.20 (VSYS)
- net VSYS: now also C18.1, U3.4 (PVDD), L5.1, U2.1 (VIN), U2.6 (EN)
- net VBUS_MAIN: now reaches U3.22 (VBUSOUT)
- net VBUS_MAIN: now also C1.1, U1.AD2 (VBUS)
- net at U3.25 (LED0): now also D3.1 (K)
- net at U3.26 (LED1): now also D2.1 (K)
- net at U3.27 (LED2): now also D1.1 (K)
- net at U3.3 (SW1): now also L6.2
- net +3V3: now reaches U3.32 (VOUT2)
- net +3V3: now also J2.1 (3V3), J3.1 (VCC), C25.1, D2.2 (A), L7.1
- net at U3.5 (SW2): now also L7.2
- net INT: now reaches U3.8 (GPIO1)
- net VBUS renamed VBUS_IN
- net VBUS_IN: now also C15.1, C24.1, D4.4 (VCC); no longer C1.1, C18.1, J2.6 (5V), U1.AD2 (VBUS)
- removed net VDDH: C19.1, C2.1, J2.1 (3V3), J3.1 (VCC), U1.Y2 (VDDH)
- new net: L5.2, U2.5 (L)
- new net: D1.2 (A), D3.2 (A)
- new net +5V: C19.1, J2.6 (5V), U2.2 (FB), U2.4 (VOUT)
- no-connect marks 6 -> 3
Other:
- note added: "5v BOOST"
- note added: "ESD"
- note added: "[x] Optional 32kHz on X1/2 [x] Figure out VDD [x] IC for power management [ ] i2c pullups [x] SWD [x] VIK [-] RESET / POWER BUTTON [x] ESD PROTECTION [x] BETTER POWER CIRCUITRY (In1.Cu = 3v3 ?) [x] BATTERY PADS [x] PROBE POINTS [x] ANT JUMPERS"
- note removed: "(global_label "VCC1" (shape input) (at 269.24 237.49 0) (fields_autoplaced) (effects (font (size 1.27 1.27)) (justify left)) (uuid 764a8019-8547-4c42-bd1d-b73854bda07f) (property "Intersheetrefs" "${INTERSHEET_REFS}" (at 277.0633 237.49 0) (effects (font (size 1.27 1.27)) (justify left) hide) ) ) (global_label "VCC1" (shape input) (at 269.24 237.49 0) (fields_autoplaced) (effects (font (size 1.27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"
- note removed: "[x] Optional 32kHz on X1/2 [x] Figure out VDD [-] IC for power management [ ] i2c pullups [x] SWD [x] VIK [-] RESET / POWER BUTTON [ ] ESD PROTECTION [ ] BETTER POWER CIRCUITRY (In1.Cu = 3v3 ?) [x] BATTERY PADS [x] PROBE POINTS [-] ANT JUMPERS"
- moved on the sheet: C10, C11, C12, C13, C9, J1, J2, J4

Commit message: almost ready for prototype 0
Parts:
- C1: footprint Connector_FFC-FPC:TE_1-84953-2_1x12-1MP_P1.0mm_Horizontal -> Capacitor_SMD:C_0603_1608Metric
- D1, D2, D3: footprint (none) -> LED_SMD:LED_0805_2012Metric
- L5, L6, L7: footprint (none) -> Inductor_SMD:L_0603_1608Metric
- R1, R2, TH1: footprint (none) -> Resistor_SMD:R_0603_1608Metric
Connections:
- net ANTENNA is gone; now on an unnamed net: J5.1 (In)
- net +3V3: now also D1.2 (A), D3.2 (A)
- net GND: now also J5.2 (Ext)
- net at C14.1, L4.1: no longer J5.2 (Ext)
Other:
- moved on the sheet: C14, J5

Commit message: benboard v0.0 r0.1
Parts:
- removed SW22: SW_Push, Button_Switch_SMD:SW_SPST_CK_KXT3, symbol Switch:SW_Push
- removed TH1: Thermistor, Resistor_SMD:R_0603_1608Metric, symbol Device:Thermistor
- added R3, R4: 47k, Resistor_SMD:R_0603_1608Metric, symbol Device:R
- added SW7: SW_DPDT, fingerpunch:SW_CuK_OS102011MA1QN1_SPDT_Angled, symbol jiran-ble:SW_DPDT
- added TP1, TP10, TP11, TP12, TP13, TP14, TP15, TP16, TP17, TP18, TP2, TP3, TP4, TP5, TP6, TP7, TP8, TP9: Probe, TestPoint:TestPoint_Pad_D1.0mm, symbol Connector:TestPoint_Probe
Connections:
- net +1V8: now also TP13.1
- net +3V3: now also R3.1, R4.1
- net D+: now also TP16.1
- net D-: now also TP17.1
- net GND: now also U3.18 (NTC)
- net MISO: now also TP8.1
- net MOSI: now also TP7.1
- net RST: now also TP11.1
- net SCK: now also R3.2, TP9.1
- net SCLK: now also TP18.1
- net SDA: now also R4.2, TP10.1
- net SPICS: now also TP4.1
- net VBAT: now also SW7.2 (B), TP14.1; no longer J4.1 (Pin_1)
- net VBUS_MAIN: now also TP12.1
- net VIK_A0: now also TP1.1
- net VIK_A1: now also TP2.1
- net VIK_RGB: now also TP3.1
- net VIK_SCL: now also TP5.1
- net VIK_SDA: now also TP6.1
- net VSYS: now also TP15.1
- new net: J4.1 (Pin_1), SW7.3 (C)
Other:
- note added: "I2C PULLUP"
- note added: "POWER MANAGEMENT"
- note added: "PROBE POINTS"
- note added: "SWITCHES"
- note added: "[x] Optional 32kHz on X1/2 [x] Figure out VDD [x] IC for power management [x] i2c pullups [x] SWD [x] VIK [x] RESET / POWER BUTTON [x] ESD PROTECTION [x] BETTER POWER CIRCUITRY (In1.Cu = 3v3 ?) [x] BATTERY PADS [x] PROBE POINTS [x] ANT JUMPERS"
- note removed: "Power Management"
- note removed: "Switches"
- note removed: "[x] Optional 32kHz on X1/2 [x] Figure out VDD [x] IC for power management [ ] i2c pullups [x] SWD [x] VIK [-] RESET / POWER BUTTON [x] ESD PROTECTION [x] BETTER POWER CIRCUITRY (In1.Cu = 3v3 ?) [x] BATTERY PADS [x] PROBE POINTS [x] ANT JUMPERS"
- moved on the sheet: C10, C11, C12, C13, C9, J4
