File: kicad/benboard.kicad_pcb (KiCad board)
At the start: 4 copper layers, 140 x 88.4 mm, 63 parts, among them J1 USB_C_Receptacle_USB2.0, J3 Conn_ARM_SWD_TagConnect_TC203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, J4 Conn_01x02_Pin, J5 Conn_Coaxial, SW1 SW_Push, SW10 SW_Push, SW11 SW_Push, SW12 SW_Push, SW13 SW_Push, SW14 SW_Push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

Commit message: this is so epic
Other:
- board text removed: "[x] SWD [x] VIK [-] RESET / POWER BUTTON [ ] ESD PROTECTION [ ] BETTER POWER CIRCUITRY (In1.Cu = 3v3) [x] BATTERY PADS [x] PROBE POINTS [-] ANT JUMPERS"
Changed lines of the file:
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@@
     (fp_line (start -6.35 -1.016) (end -6.35 -0.635)
       (stroke (width 0.15) (type solid)) (layer "B.SilkS"))
-    (fp_arc (start -2.464162 -0.61604) (mid -1.563149 -2.002043) (end 0 -2.54)
+    (fp_arc (start -2.464162 -0.61604) (mid -1.563148 -2.002044) (end 0 -2.54)
       (stroke (width 0.15) (type solid)) (layer "B.SilkS"))
     (fp_arc (start -6.35 -4.445) (mid -5.606051 -6.241051) (end -3.81 -6.985)
@@
     (fp_line (start -8.89 -1.27) (end -8.89 -3.81)
       (stroke (width 0.12) (type solid)) (layer "B.Fab"))
-    (fp_arc (start -2.464162 -0.61604) (mid -1.563149 -2.002043) (end 0 -2.54)
+    (fp_arc (start -2.464162 -0.61604) (mid -1.563148 -2.002044) (end 0 -2.54)
       (stroke (width 0.12) (type solid)) (layer "B.Fab"))
     (fp_arc (start -6.35 -4.445) (mid -5.606051 -6.241051) (end -3.81 -6.985)
@@
   (gr_line (start 120.430734 43.069228) (end 62.2 50.4)
     (stroke (width 0.1) (type default)) (layer "Edge.Cuts"))
-  (gr_text "[x] SWD\n[x] VIK\n[-] RESET / POWER BUTTON\n[ ] ESD PROTECTION\n[ ] BETTER POWER CIRCUITRY (In1.Cu = 3v3)\n[x] BATTERY PADS\n[x] PROBE POINTS\n[-] ANT JUMPERS" (at 178 180.4) (layer "Cmts.User")
-    (effects (font (size 1.5 1.5) (thickness 0.3) bold) (justify left bottom))
-  )
   (gr_text "PCB3D_TL_BENBOARD" (at 61.2 43.4) (layer "Cmts.User")
     (effects (font (size 1.5 1.5) (thickness 0.3) bold) (justify left bottom mirror))

Commit message: almost ready for prototype 0
Parts:
- removed R3, R4, R5: 10k, Resistor_SMD:R_0603_1608Metric
- removed RED1: LED, LED_SMD:LED_0805_2012Metric
- added C1: 1uF, Capacitor_SMD:C_0603_1608Metric, B.Cu at (127.0, 84.7)
- added C15: 1uF, Capacitor_SMD:C_0603_1608Metric, B.Cu at (165.9, 48.2)
- added C24: 100nF, Capacitor_SMD:C_0603_1608Metric, B.Cu at (164.4, 48.2)
- added C25: 10uF, Capacitor_SMD:C_0603_1608Metric, B.Cu at (175.6, 69.0)
- added C26: 100nF, Capacitor_SMD:C_0603_1608Metric, B.Cu at (171.9, 70.0)
- added C27: 2.2uF, Capacitor_SMD:C_0603_1608Metric, B.Cu at (165.0, 68.6)
- added D1: LED, LED_SMD:LED_0805_2012Metric, F.Cu at (155.1, 45.8)
- added D2: LED, LED_SMD:LED_0805_2012Metric, F.Cu at (152.0, 45.8)
- added D3: LED, LED_SMD:LED_0805_2012Metric, F.Cu at (149.0, 45.8)
- added D4: PRTR5V0U2X, Package_TO_SOT_SMD:SOT-143, B.Cu at (161.3, 48.7)
- added L5: 4.7uH, Inductor_SMD:L_0603_1608Metric, B.Cu at (168.6, 83.3)
- added L6: 2.2uH, Inductor_SMD:L_0603_1608Metric, B.Cu at (175.1, 65.8)
- added L7: 2.2uH, Inductor_SMD:L_0603_1608Metric, B.Cu at (175.1, 67.4)
- added TH1: Thermistor, Resistor_SMD:R_0603_1608Metric, B.Cu at (191.0, 53.2)
- added U3: nPM1300-QEXX, Package_DFN_QFN:QFN-32-1EP_5x5mm_P0.5mm_EP3.6x3.6mm_ThermalVias, B.Cu at (170.4, 66.1)
- C14, C21, J5, L4: moved to B.Cu
- C18: value 1uF -> 10uF
- C19, C20: value 4.7uF -> 10uF
- R1: value 5.1k -> 47k
- R2: value 5.1k -> 250k
- U2: value BQ24075RGT -> TPS61222DCK; footprint Package_DFN_QFN:VQFN-16-1EP_3x3mm_P0.5mm_EP1.6x1.6mm -> Package_TO_SOT_SMD:Texas_R-PDSO-G6
- moved C20 75.9 mm to (174.4, 63.6), turned to 90 degrees
- moved C18 73.9 mm to (173.8, 84.5), turned to -90 degrees
- moved C19 71.4 mm to (170.2, 86.7), turned to 180 degrees
- moved C2 68.9 mm to (171.9, 71.5), turned to 0 degrees
- moved U2 68.6 mm to (171.1, 84.5)
- moved J4 59.7 mm to (154.3, 63.8), turned to 180 degrees
- moved Y1 49.8 mm to (201.3, 90.9)
- moved C16 49.8 mm to (200.9, 88.3)
- moved C17 49.8 mm to (204.3, 91.1)
- moved C3 46.8 mm to (204.6, 80.4)
- moved C4 46.8 mm to (206.1, 80.4)
- moved L1 46.8 mm to (203.0, 82.8)
- moved L2 46.8 mm to (205.3, 82.7)
- moved R2 18.4 mm to (168.8, 70.0), turned to 180 degrees
- moved R1 17.5 mm to (166.5, 69.2)
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Connections:
- net SCL renamed VIK_SCL
- C14 pad 1: Net-(J5-Ext) -> Net-(J5-In)
- C18 pad 1: VBUS -> VSYS
- C19 pad 1: VDDH -> +5V
- C2 pad 1: VDDH -> VDD_NRF
- C20 pad 1: VBAT -> VDD_NRF
- J1 pad A4: VBUS -> VBUS_IN
- J1 pad A5: Net-(J1-CC1) -> CC1
- J1 pad A9: VBUS -> VBUS_IN
- J1 pad B4: VBUS -> VBUS_IN
- J1 pad B5: Net-(J1-CC2) -> CC2
- J1 pad B9: VBUS -> VBUS_IN
- J2 pad 1: VDDH -> +3V3
- J2 pad 3: SDA -> VIK_SDA
- J2 pad 6: VBUS -> +5V
- J3 pad 1: VDDH -> +3V3
- J5 pad 1: ANTENNA -> Net-(J5-In)
- J5 pad 2: Net-(J5-Ext) -> GND
- L4 pad 1: Net-(J5-Ext) -> Net-(J5-In)
- R1 pad 1: Net-(J1-CC1) -> Net-(U3-VSET1)
- R2 pad 1: Net-(J1-CC2) -> GND
- R2 pad 2: GND -> Net-(U3-VSET2)
- U1 pad AD2: VBUS -> VBUS_MAIN
- U1 pad AD8: POWER -> unconnected-(U1-P0.13-PadAD8)
- U1 pad B19: SDA -> VIK_SDA
- U1 pad J1: unconnected-(U1-AIN2/P0.04-PadJ1) -> SDA
- U1 pad K2: unconnected-(U1-AIN3/P0.05-PadK2) -> SCK
- U1 pad Y2: VDDH -> VDD_NRF
- U2 pad 1: Net-(U2-TS) -> VSYS
- U2 pad 2: VBAT -> +5V
- U2 pad 3: VBAT -> GND
- U2 pad 4: GND -> +5V
- U2 pad 5: GND -> Net-(U2-L)
- U2 pad 6: VDDH -> VSYS
Routing:
- net VBUS: track 187.6 -> 0.00 mm, vias 5 -> 0
- net +3V3: track 0.00 -> 113.5 mm, vias 0 -> 3
- net VDDH: track 85.2 -> 0.00 mm, vias 6 -> 0
- net VDD_NRF: track 32.4 -> 91.6 mm, vias 5 -> 7
- net Net-(RED1-K): track 56.7 -> 0.00 mm, vias 4 -> 0
- net SCK: track 0.00 -> 56.0 mm, vias 0 -> 6
- net VIK_SDA: track 0.00 -> 55.4 mm, vias 0 -> 2
- net VBUS_IN: track 0.00 -> 51.2 mm, vias 0 -> 2
- net VBUS_MAIN: track 0.00 -> 47.6 mm, vias 0 -> 2
- net CC2: track 0.00 -> 42.4 mm, vias 0 -> 2
- net CC1: track 0.00 -> 40.9 mm, vias 0 -> 2
- net VSYS: track 0.00 -> 38.1 mm, vias 0 -> 2
- net +5V: track 0.00 -> 37.7 mm, vias 0 -> 2
- net Net-(D3-K): track 0.00 -> 37.1 mm, vias 0 -> 2
- net Net-(D2-K): track 0.00 -> 34.7 mm, vias 0 -> 2
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
Commit message: benboard v0.0 r0.1
Parts:
- removed TH1: Thermistor, Resistor_SMD:R_0603_1608Metric
- added G***: LOGO, LOGO, F.Cu at (127.4, 87.7)
- added R3: 47k, Resistor_SMD:R_0603_1608Metric, B.Cu at (160.7, 70.9)
- added R4: 47k, Resistor_SMD:R_0603_1608Metric, B.Cu at (162.2, 71.0)
- added REF**: MountingHole_2.2mm_M2, MountingHole:MountingHole_2.2mm_M2, F.Cu at (199.6, 113.7)
- added REF**: MountingHole_2.2mm_M2, MountingHole:MountingHole_2.2mm_M2, F.Cu at (64.3, 109.0)
- added REF**: MountingHole_2.2mm_M2, MountingHole:MountingHole_2.2mm_M2, F.Cu at (176.6, 105.0)
- added REF**: MountingHole_2.2mm_M2, MountingHole:MountingHole_2.2mm_M2, F.Cu at (195.4, 128.8)
- added REF**: MountingHole_2.2mm_M2, MountingHole:MountingHole_2.2mm_M2, F.Cu at (140.4, 121.3)
- added REF**: MountingHole_2.2mm_M2, MountingHole:MountingHole_2.2mm_M2, F.Cu at (119.4, 82.5)
- added REF**: MountingHole_2.2mm_M2, MountingHole:MountingHole_2.2mm_M2, F.Cu at (120.3, 45.4)
- added REF**: MountingHole_2.2mm_M2, MountingHole:MountingHole_2.2mm_M2, F.Cu at (176.3, 52.5)
- added REF**: MountingHole_2.2mm_M2, MountingHole:MountingHole_2.2mm_M2, F.Cu at (146.3, 45.3)
- added REF**: MountingHole_2.2mm_M2, MountingHole:MountingHole_2.2mm_M2, F.Cu at (163.3, 84.1)
- added REF**: MountingHole_2.2mm_M2, MountingHole:MountingHole_2.2mm_M2, F.Cu at (64.2, 52.2)
- added REF**: MountingHole_2.2mm_M2, MountingHole:MountingHole_2.2mm_M2, F.Cu at (81.8, 72.3)
- added REF**: MountingHole_2.2mm_M2, MountingHole:MountingHole_2.2mm_M2, F.Cu at (87.0, 108.9)
- added TP1: Probe, TestPoint:TestPoint_Pad_D1.0mm, B.Cu at (183.8, 109.7)
- added TP10: Probe, TestPoint:TestPoint_Pad_D1.0mm, B.Cu at (160.3, 75.8)
- added TP11: Probe, TestPoint:TestPoint_Pad_D1.0mm, B.Cu at (142.7, 71.2)
- added TP12: Probe, TestPoint:TestPoint_Pad_D1.0mm, B.Cu at (160.7, 68.3)
- added TP13: Probe, TestPoint:TestPoint_Pad_D1.0mm, B.Cu at (176.2, 63.2)
- added TP14: Probe, TestPoint:TestPoint_Pad_D1.0mm, B.Cu at (163.0, 67.8)
- added TP15: Probe, TestPoint:TestPoint_Pad_D1.0mm, B.Cu at (164.8, 72.7)
- added TP16: Probe, TestPoint:TestPoint_Pad_D1.0mm, B.Cu at (173.5, 53.0)
- added TP17: Probe, TestPoint:TestPoint_Pad_D1.0mm, B.Cu at (171.4, 53.0)
- added TP18: Probe, TestPoint:TestPoint_Pad_D1.0mm, B.Cu at (184.6, 114.8)
- added TP2: Probe, TestPoint:TestPoint_Pad_D1.0mm, B.Cu at (179.3, 117.1)
- added TP3: Probe, TestPoint:TestPoint_Pad_D1.0mm, B.Cu at (176.6, 107.4)
- added TP4: Probe, TestPoint:TestPoint_Pad_D1.0mm, B.Cu at (181.3, 117.2)
- added TP5: Probe, TestPoint:TestPoint_Pad_D1.0mm, B.Cu at (178.4, 109.1)
- added TP6: Probe, TestPoint:TestPoint_Pad_D1.0mm, B.Cu at (181.8, 108.8)
- added TP7: Probe, TestPoint:TestPoint_Pad_D1.0mm, B.Cu at (173.7, 114.1)
- added TP8: Probe, TestPoint:TestPoint_Pad_D1.0mm, B.Cu at (183.3, 117.1)
- added TP9: Probe, TestPoint:TestPoint_Pad_D1.0mm, B.Cu at (160.3, 73.6)
- SW22: value SW_Push -> SW_DPDT; footprint Button_Switch_SMD:SW_SPST_CK_KXT3 -> fingerpunch:SW_CuK_OS102011MA1QN1_SPDT_Angled; moved to B.Cu
- moved C3 50.8 mm to (153.9, 84.9), turned to -90 degrees
- moved L2 50.6 mm to (154.7, 82.6), turned to 0 degrees
- moved C4 50.0 mm to (156.2, 84.1), turned to 0 degrees
- moved L1 48.4 mm to (154.7, 81.1), turned to 180 degrees
- moved C16 47.1 mm to (153.8, 87.8), turned to 0 degrees
- moved C17 43.9 mm to (160.6, 86.9)
- moved Y1 43.9 mm to (157.6, 86.7)
- moved D1 10.9 mm to (166.0, 45.6)
- moved D2 10.9 mm to (162.9, 45.6)
- moved D3 10.9 mm to (159.9, 45.6)
- moved C1 10.6 mm to (136.3, 79.6), turned to -90 degrees
- moved C7 7.68 mm to (150.7, 86.8), turned to 0 degrees
- moved SW22 7.06 mm to (151.5, 45.3), turned to 0 degrees
- moved C5 0.59 mm to (134.0, 80.4)
Connections:
- J4 pad 1: VBAT -> Net-(J4-Pin_1)
- SW22 pad 1: GND -> unconnected-(SW22-A-Pad1)
- SW22 pad 2: RST -> VBAT
Routing:
- net RST: track 1.61 -> 69.7 mm, vias 1 -> 4
- net VBAT: track 17.5 -> 71.9 mm, vias 1 -> 3
- net Net-(J4-Pin_1): track 0.00 -> 52.6 mm
- net Net-(U1-DEC4): track 8.97 -> 31.3 mm, vias 2 -> 3
- net +3V3: track 113.5 -> 135.1 mm, vias 3 -> 4
- net Net-(U1-XC2): track 0.00 -> 20.7 mm, vias 0 -> 2
- net Net-(U1-XC1): track 0.00 -> 20.0 mm, vias 0 -> 2
- net Net-(U1-DCC): track 8.36 -> 25.1 mm, vias 1 -> 2
- net Net-(U1-DEC3): track 1.49 -> 10.6 mm
- net VIK_RGB: track 57.5 -> 66.1 mm, vias 2 -> 4
- net MOSI: track 60.9 -> 69.2 mm, vias 0 -> 2
- net SDA: track 64.4 -> 72.3 mm, vias 4 -> 5
- net D-: track 74.9 -> 81.5 mm, vias 3 -> 4
- net Net-(D3-K): track 37.1 -> 30.7 mm
- net VIK_A1: track 62.7 -> 68.9 mm, vias 2 -> 4
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Other:
- board text added: "+"
- board text added: "-"
- board text added: "JLCJLCJLCJLC"

Commit message: that's it now i SWEAR
Parts:
- added G***: LOGO, LOGO, B.Cu at (115.1, 104.5)
- added G***: LOGO, LOGO, B.Cu at (104.0, 104.4)
- added G***: LOGO, LOGO, B.Cu at (109.2, 104.2)
- added G***: LOGO, LOGO, B.Cu at (149.3, 107.2)
- moved G*** 2.75 mm to (162.3, 108.3)
